File: rp2354.kicad_pcb (KiCad board)
At the start: 2 copper layers, 41 parts, among them J1 Conn_01x20_Pin, J2 USB_C_Receptacle_USB2.0_16P, J4 Conn_01x20_Pin, SW1 SW_SPST, SW2 SW_SPST, U1 RP2354A, U4 TMI3112H, Y2 Crystal_GND24_Small

Commit message: July25
Parts:
- moved R10 35.6 mm to (178.8, 128.9), turned to 90 degrees
- moved SW2 31.3 mm to (181.6, 127.6), turned to 90 degrees
- moved Y2 10.8 mm to (185.3, 130.5)
- moved C13 9.05 mm to (183.3, 117.2), turned to -90 degrees
- moved D2 6.81 mm to (181.2, 122.4)
- moved R9 6.73 mm to (183.7, 121.5)
- moved R8 6.68 mm to (191.0, 94.3)
- moved C14 6.52 mm to (183.0, 123.9)
- moved J1 6.38 mm to (195.1, 131.5)
- moved C19 6.04 mm to (181.8, 98.5), turned to 90 degrees
- moved J4 5.19 mm to (174.8, 83.3)
- moved SW1 5.06 mm to (189.0, 127.6), turned to 90 degrees
- moved C21 4.45 mm to (188.0, 115.9), turned to -90 degrees
- moved C16 3.97 mm to (191.7, 108.7)
- moved C24 3.46 mm to (184.8, 96.0)
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Routing:
- net GPIO16: track 0.00 -> 27.7 mm
- net GPIO0: track 0.00 -> 25.0 mm
- net GPIO15: track 0.00 -> 25.0 mm
- net GPIO17: track 0.00 -> 24.2 mm
- net GPIO1: track 0.00 -> 23.1 mm
- net Net-(SW2-B): track 12.0 -> 34.1 mm, vias 0 -> 2
- net GPIO14: track 0.00 -> 21.6 mm
- net GPIO29_ADC3: track 0.00 -> 20.2 mm, vias 0 -> 2
- net GPIO13: track 0.00 -> 19.9 mm
- net GPIO28_ADC2: track 0.00 -> 19.7 mm
- net GPIO2: track 0.00 -> 19.4 mm
- net GPIO18: track 0.00 -> 18.6 mm
- net GPIO12: track 0.00 -> 18.3 mm
- net GPIO27_ADC1: track 0.00 -> 17.8 mm
- net GPIO3: track 0.00 -> 17.4 mm
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