File: rp2354.kicad_sch (KiCad schematic)
At the start: 42 parts, among them J1 Conn_01x20_Pin, J2 USB_C_Receptacle_USB2.0_16P, J4 Conn_01x20_Pin, J6 Conn_01x03_Pin, SW1 SW_SPST, SW2 SW_SPST, U1 RP2354A, U4 TMI3112H, Y2 Crystal_GND24_Small

Commit message: July25
Other:
- moved on the sheet: R9
Changed lines of the file:
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@@
 	(wire
 		(pts
+			(xy 259.08 92.71) (xy 257.81 92.71)
+		)
+		(stroke
+			(width 0)
+			(type default)
+		)
+	)
+	(wire
+		(pts
 			(xy 224.79 100.33) (xy 231.14 100.33)
 		)
@@
 	(wire
 		(pts
+			(xy 266.7 92.71) (xy 265.43 92.71)
+		)
+		(stroke
+			(width 0)
+			(type default)
+		)
+	)
+	(wire
+		(pts
 			(xy 81.28 43.18) (xy 83.82 43.18)
 		)
@@
 	(symbol
 		(lib_id "Device:R")
-		(at 261.62 92.71 90)
+		(at 262.89 92.71 90)
 		(unit 1)
 		(exclude_from_sim no)
@@
 		(dnp no)
 		(property "Reference" "R9"
-			(at 261.62 86.36 90)
+			(at 262.89 86.36 90)
 			(effects
 				(font
@@
 		)
 		(property "Value" "33k2"
-			(at 261.62 88.9 90)
+			(at 262.89 88.9 90)
 			(effects
 				(font
@@
 		)
 		(property "Footprint" "Resistor_SMD:R_0603_1608Metric"
-			(at 261.62 94.488 90)
+			(at 262.89 94.488 90)
 			(effects
 				(font
@@
 		)
 		(property "Datasheet" "~"
-			(at 261.62 92.71 0)
+			(at 262.89 92.71 0)
 			(effects
 				(font
@@
 		)
 		(property "Description" "Resistor"
-			(at 261.62 92.71 0)
+			(at 262.89 92.71 0)
 			(effects
 				(font
